File: Hardware/Proiect TSC.brd (EAGLE design)
At the start: 46 x 35 mm, 105 parts, among them IC1 BQ25180YBGR, IC2 RT6160AWSC, IC3 BMA423, IC4 DRV2605YZFR, J1 TC2030-IDC, J2 503480-2400, J3 KH-TYPE-C-16P, Q1 20V/4.2A/52mΩ/1.4W, Q2 SI1308EDL, SW1 SW1, SW2 2025-10-22_07-23-44_LIBRARY_E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, SW3 2025-10-22_07-23-44_LIBRARY_E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, U1 MAX17048G+T10, U2 NRF52840_QF, X1 32MHz, X2 32.768kHz

Commit message: WIP commit. Still adding features
Signed-off-by: Teodor Panait <teodordpanait@gmail.com>
Parts:
- moved TP_GND 40.2 mm to (-54.1, 117.9)
- moved TP_3.3V 38.7 mm to (-92.1, 124.4)
- moved C28 34.5 mm to (-89.6, 122.9), turned to 0 degrees
- moved TP_SCL 33.4 mm to (-54.8, 122.3)
- moved TP_SDA 31.0 mm to (-56.3, 123.9)
- moved C11 29.5 mm to (-68.0, 110.9), turned to 0 degrees
- moved TP_VBAT 25.0 mm to (-93.3, 122.5)
- moved X2 24.8 mm to (-70.2, 113.3)
- moved TP_RESET 24.1 mm to (-53.9, 115.5)
- moved C13 22.6 mm to (-88.4, 125.2), turned to 90 degrees
- moved C10 22.2 mm to (-69.8, 114.9), turned to 0 degrees
- moved U$39 21.4 mm to (-77.8, 118.4), turned to 0 degrees
- moved U$38 20.8 mm to (-77.6, 119.3), turned to 0 degrees
- moved C9 19.1 mm to (-85.8, 123.5), turned to 270 degrees
- moved C36 18.2 mm to (-88.5, 95.8)
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Connections:
- net ALERT/1.6C renamed ALERT
- net P0.14/2.7C renamed P0.14
- removed net 3V3/1.7D: C33.1, IC4.C2, Q1.2, R11.2, R12.2, R13.2, R7.2
- removed net 3V3/2.4A: C13.1, C17.1, C26.1, C28.1, C29.1, C5.1, C6.1, C9.1, IC2.E2, IC2.E3, IC3.10, IC3.3, IC3.7, J1.1, R2.1, R3.1, TP_3.3V.TP, TP_3V3.TP, U2.P$A22, U2.P$AD14, U2.P$AD23, U2.P$B1, U2.P$W1, U2.P$Y2
- removed net D+/1.5D: D1.4
- removed net D+/2.7D: U2.P$AD6
- removed net D-/1.5D: D1.6
- removed net D-/2.7D: U2.P$AD4
- removed net EPD_BUSY/1.5C: J2.9
- removed net EPD_BUSY/2.2D: U2.P$AD12
- removed net EPD_CS/1.4C: J2.12
- removed net EPD_CS/2.2D: U2.P$K2
- removed net EPD_DC/1.5D: J2.11
- removed net EPD_DC/2.2D: U2.P$AD10
- removed net EPD_RST/1.5D: J2.10
- removed net EPD_RST/2.2D: U2.P$AC11
- removed net HAPTIC_EN/1.4C: IC4.A1
- removed net HAPTIC_EN/2.6A: U2.P$U1
- removed net MOSI/1.5B: J2.14
- removed net MOSI/2.2D: U2.P$B13
- removed net P0.13/1.5D: C36.1, R11.1, SW1.2
- removed net P0.13/2.6C: U2.P$AD8
- removed net P1.01/1.6C: Q1.1, R7.1
- removed net P1.01/2.4B: U2.P$Y23
- removed net P1.02/1.6C: C34.1, R13.1, SW3.2
- removed net P1.02/2.8C: U2.P$W24
- removed net P1.14/1.5D: C35.1, R12.1, SW2.2
- removed net SCK/1.5B: J2.13
- removed net SCK/2.2D: U2.P$A12
- removed net SCL/1.4C: IC4.C1, U1.7
- removed net SCL/2.4C: IC1.B1, IC3.12, R2.2, R4.2, TP_SCL.TP, U2.P$M2
- removed net SDA/1.4C: IC4.B2, U1.8
- removed net SDA/2.4C: IC1.C1, IC3.2, R3.2, R5.2, TP_SDA.TP, U2.P$L1
- removed net VBAT/1.2A: C37.1, TP_VBAT.TP, U1.2, U1.3
- removed net VBAT/2.5C: C3.1, IC1.C2
- removed net VBUS/1.5D: D1.5, J3.A4_B9, J3.A9_B4, U$38.1, U$39.1
- removed net VBUS/2.6D: C1.1, C7.1, IC1.A2, U2.P$AD2
- new net 3V3: C13.1, C17.1, C26.1, C28.1, C29.1, C33.1, C5.1, C6.1, C9.1, IC2.E2, IC2.E3, IC3.10, IC3.3, IC3.7, IC4.C2, J1.1, Q1.2, R11.2, R12.2, R13.2, R2.1, R3.1, R7.2, TP_3.3V.TP, TP_3V3.TP, U2.P$A22, U2.P$AD14, U2.P$AD23, U2.P$B1, U2.P$W1, U2.P$Y2
- new net D+: D1.4, U2.P$AD6
- new net D-: D1.6, U2.P$AD4
- new net EPD_BUSY: J2.9, U2.P$AD12
- new net EPD_CS: J2.12, U2.P$K2
- new net EPD_DC: J2.11, U2.P$AD10
- new net EPD_RST: J2.10, U2.P$AC11
- new net HAPTIC_EN: IC4.A1, U2.P$U1
- new net MOSI: J2.14, U2.P$B13
- new net P0.13: C36.1, R11.1, SW1.2, U2.P$AD8
- new net P1.01: Q1.1, R7.1, U2.P$Y23
- new net P1.02: C34.1, R13.1, SW3.2, U2.P$W24
- new net SCK: J2.13, U2.P$A12
- new net SCL: IC1.B1, IC3.12, IC4.C1, R2.2, R4.2, TP_SCL.TP, U1.7, U2.P$M2
- new net SDA: IC1.C1, IC3.2, IC4.B2, R3.2, R5.2, TP_SDA.TP, U1.8, U2.P$L1
- new net VBAT: C3.1, C37.1, IC1.C2, TP_VBAT.TP, U1.2, U1.3
- new net VBUS: C1.1, C7.1, D1.5, IC1.A2, J3.A4_B9, J3.A9_B4, U$38.1, U$39.1, U2.P$AD2
- net P1.14: now also C35.1, R12.1, SW2.2
Routing:
- net 3V3: track 0.00 -> 150.1 mm, vias 0 -> 10
- net 3V3/2.4A: track 121.1 -> 0.00 mm, vias 7 -> 0
- net 3V3/1.7D: track 58.4 -> 0.00 mm, vias 4 -> 0
- net VBAT: track 0.00 -> 57.0 mm
- net SDA: track 0.00 -> 52.3 mm, vias 0 -> 8
- net SCL: track 0.00 -> 49.4 mm, vias 0 -> 5
- net P1.14: track 0.00 -> 44.0 mm, vias 0 -> 4
- net VREG: track 57.6 -> 15.4 mm, vias 4 -> 0
- net P0.13: track 0.00 -> 41.4 mm
- net SCL/2.4C: track 40.1 -> 0.00 mm, vias 3 -> 0
- net VBUS/2.6D: track 38.1 -> 0.00 mm, vias 2 -> 0
- net SDA/2.4C: track 37.9 -> 0.00 mm, vias 4 -> 0
- net HAPTIC_EN: track 0.00 -> 34.5 mm, vias 0 -> 2
- net GND: track 298.3 -> 264.9 mm, vias 7 -> 5
- net P1.02: track 0.00 -> 23.2 mm, vias 0 -> 3
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