File: Hardware/Proiect_TSC.sch (EAGLE design)
At the start: 105 parts, among them IC1 BQ25180YBGR, IC2 RT6160AWSC, IC3 BMA423, IC4 DRV2605YZFR, J1 TC2030-IDC, J2 503480-2400, J3 KH-TYPE-C-16P, Q1 20V/4.2A/52mΩ/1.4W, Q2 SI1308EDL, SW1 SW1, SW2 2025-10-22_07-23-44_LIBRARY_E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, SW3 2025-10-22_07-23-44_LIBRARY_E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, U1 MAX17048G+T10, U2 NRF52840_QF, X1 32MHz, X2 32.768kHz

Commit message: WIP commit. Still adding features
Signed-off-by: Teodor Panait <teodordpanait@gmail.com>
Connections:
- net ALERT/1.6C renamed ALERT
- net P0.14/2.7C renamed P0.14
- removed net 3V3/1.7D: C33.1, IC4.VDD, Q1.S, R11.2, R12.2, R13.2, R7.2
- removed net 3V3/2.4A: C13.1, C17.1, C26.1, C28.1, C29.1, C5.1, C6.1, C9.1, IC2.VOUT_1, IC2.VOUT_2, IC3.CSB, IC3.VDD, IC3.VDDIO, J1.1, R2.1, R3.1, TP_3.3V.TP, TP_3V3.TP, U2.VDD@A22, U2.VDD@AD14, U2.VDD@AD23, U2.VDD@B1, U2.VDD@W1, U2.VDDH@Y2
- removed net D+/1.5D: D1.I/O2_2
- removed net D+/2.7D: U2.D+@AD6
- removed net D-/1.5D: D1.I/O1_2
- removed net D-/2.7D: U2.D-@AD4
- removed net EPD_BUSY/1.5C: J2.9
- removed net EPD_BUSY/2.2D: U2.P0.17@AD12
- removed net EPD_CS/1.4C: J2.12
- removed net EPD_CS/2.2D: U2.P0.05/AIN3@K2
- removed net EPD_DC/1.5D: J2.11
- removed net EPD_DC/2.2D: U2.P0.15@AD10
- removed net EPD_RST/1.5D: J2.10
- removed net EPD_RST/2.2D: U2.P0.16@AC11
- removed net HAPTIC_EN/1.4C: IC4.EN
- removed net HAPTIC_EN/2.6A: U2.P0.12@U1
- removed net MOSI/1.5B: J2.14
- removed net MOSI/2.2D: U2.P0.03/AIN1@B13
- removed net P0.13/1.5D: C36.1, R11.1, SW1.2
- removed net P0.13/2.6C: U2.P0.13@AD8
- removed net P1.01/1.6C: Q1.G, R7.1
- removed net P1.01/2.4B: U2.P1.01@Y23
- removed net P1.02/1.6C: C34.1, R13.1, SW3.2
- removed net P1.02/2.8C: U2.P1.02@W24
- removed net P1.14/1.5D: C35.1, R12.1, SW2.2
- removed net SCK/1.5B: J2.13
- removed net SCK/2.2D: U2.P0.02/AIN0@A12
- removed net SCL/1.4C: IC4.SCL, U1.SCL
- removed net SCL/2.4C: IC1.SCL, IC3.SCX, R2.2, R4.2, TP_SCL.TP, U2.P0.07@M2
- removed net SDA/1.4C: IC4.SDA, U1.SDA
- removed net SDA/2.4C: IC1.SDA, IC3.SDX, R3.2, R5.2, TP_SDA.TP, U2.P0.06@L1
- removed net VBAT/1.2A: C37.1, TP_VBAT.TP, U1.CELL, U1.VDD
- removed net VBAT/2.5C: C3.1, IC1.BAT
- removed net VBUS/1.5D: D1.VBUS, J3.VBUS, U$38.1, U$39.1
- removed net VBUS/2.6D: C1.1, C7.1, IC1.IN, U2.VBUS@AD2
- new net 3V3: C13.1, C17.1, C26.1, C28.1, C29.1, C33.1, C5.1, C6.1, C9.1, IC2.VOUT_1, IC2.VOUT_2, IC3.CSB, IC3.VDD, IC3.VDDIO, IC4.VDD, J1.1, Q1.S, R11.2, R12.2, R13.2, R2.1, R3.1, R7.2, TP_3.3V.TP, TP_3V3.TP, U2.VDD@A22, U2.VDD@AD14, U2.VDD@AD23, U2.VDD@B1, U2.VDD@W1, U2.VDDH@Y2
- new net D+: D1.I/O2_2, U2.D+@AD6
- new net D-: D1.I/O1_2, U2.D-@AD4
- new net EPD_BUSY: J2.9, U2.P0.17@AD12
- new net EPD_CS: J2.12, U2.P0.05/AIN3@K2
- new net EPD_DC: J2.11, U2.P0.15@AD10
- new net EPD_RST: J2.10, U2.P0.16@AC11
- new net HAPTIC_EN: IC4.EN, U2.P0.12@U1
- new net MOSI: J2.14, U2.P0.03/AIN1@B13
- new net P0.13: C36.1, R11.1, SW1.2, U2.P0.13@AD8
- new net P1.01: Q1.G, R7.1, U2.P1.01@Y23
- new net P1.02: C34.1, R13.1, SW3.2, U2.P1.02@W24
- new net SCK: J2.13, U2.P0.02/AIN0@A12
- new net SCL: IC1.SCL, IC3.SCX, IC4.SCL, R2.2, R4.2, TP_SCL.TP, U1.SCL, U2.P0.07@M2
- new net SDA: IC1.SDA, IC3.SDX, IC4.SDA, R3.2, R5.2, TP_SDA.TP, U1.SDA, U2.P0.06@L1
- new net VBAT: C3.1, C37.1, IC1.BAT, TP_VBAT.TP, U1.CELL, U1.VDD
- new net VBUS: C1.1, C7.1, D1.VBUS, IC1.IN, J3.VBUS, U$38.1, U$39.1, U2.VBUS@AD2
- net P1.14: now also C35.1, R12.1, SW2.2
Other:
- note added: "Buttons"
- note added: "E-Paper display connector"
- note added: "E-paper drive circuit"
- note added: "Fuel Gauge"
- note added: "Haptic Driver"
- note added: "IMU"
- note added: "Panait Teodor-Dimitrie"
- note added: "SWD"
- note added: "USB-C Connector and ESD Protection"
